Commit message: gps fusion

File: jackal/jackal_description/urdf/accessories.urdf.xacro (robot description, xacro)
@@ -380,18 +380,4 @@
     </xacro:unless>
   </xacro:if>
-  <!-- BlackflyS Camera -->
-  <xacro:if value="$(optenv JACKAL_BLACKFLY 0)">
-    <xacro:include filename="$(find flir_camera_description)/urdf/flir_blackflys.urdf.xacro"/>
-    <xacro:property name="prefix" value="$(optenv JACKAL_BLACKFLY_PREFIX front_camera)"/>
-    <xacro:property name="parent" value="$(optenv JACKAL_BLACKFLY_PARENT front_mount)"/>
-    <xacro:property name="xyz"    value="$(optenv JACKAL_BLACKFLY_OFFSET 0 0 0)"/>
-    <xacro:property name="rpy"    value="$(optenv JACKAL_BLACKFLY_RPY    0 0 0)"/>
-    <xacro:flir_blackflys frame="${prefix}"/>
-    <joint name="${prefix}_mount_joint" type="fixed">
-      <child link="${prefix}"/>
-      <parent link="${parent}"/>
-      <origin xyz="${xyz}" rpy="${rpy}" />
-    </joint>
-  </xacro:if>
   <!-- Fender Accessories -->
   <xacro:if value="$(optenv JACKAL_FRONT_ACCESSORY_FENDER 0)">
