Commit message: edited

File: jackal/jackal_description/urdf/mass.urdf.xacro (robot description, xacro)
@@ -14,5 +14,5 @@
   <xacro:property name="stretcher_width" value="0.620" />
   <xacro:property name="stretcher_height" value="0.05" />
-  <xacro:property name="stretcher_mount_dist" value="0.05" />
+  <xacro:property name="stretcher_mount_dist" value="0.10" />
   <xacro:property name="dummy_inertia" value="1e-09"/>
   <xacro:property name="mount_spacing" value="0.120" />
@@ -206,19 +206,26 @@
   </joint>
   <!-- Stretcher -->
-  <link name="base_stretcher">
+  <link name="base_stretcher_link">
     <visual>
       <geometry>
         <box size="${stretcher_length} ${stretcher_width} ${stretcher_height}" />
       </geometry>
+      <origin xyz="0 0 0" />
       <material name="navy" />
     </visual>
+    <collision>
+      <origin xyz="0 0 0" />
+      <geometry>
+        <box size="${stretcher_length} ${stretcher_width} ${stretcher_height}" />
+      </geometry>
+    </collision>
   </link>
   <joint name="base_stretcher_joint" type="fixed">
     <parent link="chassis_link" />
-    <child link="base_stretcher" />
+    <child link="base_stretcher_link" />
     <origin xyz="0 0 ${chassis_height + stretcher_mount_dist}" />
   </joint>
   <xacro:macro name="handle" params="prefix reflect">
-    <link name="${prefix}_handle">
+    <link name="${prefix}_handle_link">
       <visual>
         <geometry>
@@ -228,10 +235,20 @@
         <material name="light_grey" />
       </visual>
+      <collision>
+        <origin xyz="0 0 0" rpy="0 ${PI/2} 0"/>
+        <geometry>
+          <cylinder length="${stretcher_length+0.5}" radius="${stretcher_height/2}"/>
+        </geometry>
+      </collision>
     </link>
     <joint name="${prefix}_handle_joint" type="fixed">
-        <parent link="base_stretcher"/>
-        <child link="${prefix}_handle"/>
+        <parent link="base_stretcher_link"/>
+        <child link="${prefix}_handle_link"/>
         <origin xyz="0 ${reflect*(stretcher_width/2 + stretcher_height/2)} ${stretcher_height/4}" />
     </joint>
+    <gazebo reference="${prefix}_handle_link">
+      <material>Gazebo/White</material>
+      <selfCollide>false</selfCollide>
+    </gazebo>
   </xacro:macro>
   <xacro:handle prefix="right" reflect="1" />
@@ -256,5 +273,5 @@
   </joint>
   <!-- Bring in simulation data for Gazebo. -->
-  <xacro:include filename="$(find jackal_description)/urdf/jackal.gazebo" />
+  <xacro:include filename="$(find jackal_description)/urdf/mass.gazebo" />
   <!-- Optional standard accessories, including their simulation data. The rendering
        of these into the final description is controlled by optenv variables, which

Commit message: added supports

File: jackal/jackal_description/urdf/mass.urdf.xacro (robot description, xacro)
@@ -14,5 +14,5 @@
   <xacro:property name="stretcher_width" value="0.620" />
   <xacro:property name="stretcher_height" value="0.05" />
-  <xacro:property name="stretcher_mount_dist" value="0.10" />
+  <xacro:property name="stretcher_mount_dist" value="0.216" />
   <xacro:property name="dummy_inertia" value="1e-09"/>
   <xacro:property name="mount_spacing" value="0.120" />
@@ -211,9 +211,9 @@
         <box size="${stretcher_length} ${stretcher_width} ${stretcher_height}" />
       </geometry>
-      <origin xyz="0 0 0" />
+      <origin xyz="0 0 ${stretcher_mount_dist}" />
       <material name="navy" />
     </visual>
     <collision>
-      <origin xyz="0 0 0" />
+      <origin xyz="0 0 ${stretcher_mount_dist}" />
       <geometry>
         <box size="${stretcher_length} ${stretcher_width} ${stretcher_height}" />
@@ -224,7 +224,7 @@
     <parent link="chassis_link" />
     <child link="base_stretcher_link" />
-    <origin xyz="0 0 ${chassis_height + stretcher_mount_dist}" />
-  </joint>
-  <xacro:macro name="handle" params="prefix reflect">
+    <origin xyz="0 0 ${chassis_height}" />
+  </joint>
+  <xacro:macro name="stretcher_handle" params="prefix reflect">
     <link name="${prefix}_handle_link">
       <visual>
@@ -232,9 +232,9 @@
           <cylinder length="${stretcher_length+0.5}" radius="${stretcher_height/2}"/>
         </geometry>
-        <origin xyz="0 0 0" rpy="0 ${PI/2} 0"/>
+        <origin xyz="0 0 ${stretcher_mount_dist}" rpy="0 ${PI/2} 0"/>
         <material name="light_grey" />
       </visual>
       <collision>
-        <origin xyz="0 0 0" rpy="0 ${PI/2} 0"/>
+        <origin xyz="0 0 ${stretcher_mount_dist}" rpy="0 ${PI/2} 0"/>
         <geometry>
           <cylinder length="${stretcher_length+0.5}" radius="${stretcher_height/2}"/>
@@ -252,6 +252,34 @@
     </gazebo>
   </xacro:macro>
-  <xacro:handle prefix="right" reflect="1" />
-  <xacro:handle prefix="left" reflect="-1" />
+  <xacro:stretcher_handle prefix="right" reflect="1" />
+  <xacro:stretcher_handle prefix="left" reflect="-1" />
+  <xacro:macro name="stretcher_support" params="prefix x_offset y_offset z_offset">
+    <link name="${prefix}_support_link">
+      <visual>
+        <geometry>
+          <cylinder length="${stretcher_mount_dist}" radius="0.02" />
+        </geometry>
+        <origin xyz="0 0 0" rpy="0 0 0" />
+        <material name="light_grey" />
+      </visual>
+      <collision>
+        <origin xyz="0 0 0" rpy="0 0 0" />
+        <geometry>
+          <cylinder length="${stretcher_mount_dist}" radius="0.02" />
+        </geometry>
+      </collision>
+    </link>
+    <joint name="${prefix}_support_joint" type="fixed">
+      <parent link="chassis_link" />
+      <child link="${prefix}_support_link" />
+      <origin xyz="${x_offset} ${y_offset} ${z_offset}" rpy="0 0 0" />
+    </joint>
+  </xacro:macro>
+  <!-- Front right and left supports -->
+  <xacro:stretcher_support prefix="front_right" x_offset="${mount_spacing}" y_offset="${stretcher_width/5}" z_offset="${chassis_height/2 * 3}" />
+  <xacro:stretcher_support prefix="front_left" x_offset="${mount_spacing}" y_offset="${-stretcher_width/5}" z_offset="${chassis_height/2 * 3}" />
+  <!-- Rear right and left supports -->
+  <xacro:stretcher_support prefix="rear_right" x_offset="${-mount_spacing}" y_offset="${stretcher_width/5}" z_offset="${chassis_height/2 * 3}" />
+  <xacro:stretcher_support prefix="rear_left" x_offset="${-mount_spacing}" y_offset="${-stretcher_width/5}" z_offset="${chassis_height/2 * 3}" />
   <link name="mid_mount"></link>
   <joint name="mid_mount_joint" type="fixed">

Commit message: final commit

File: jackal/jackal_description/urdf/mass.urdf.xacro (robot description, xacro)
@@ -258,5 +258,5 @@
       <visual>
         <geometry>
-          <cylinder length="${stretcher_mount_dist}" radius="0.02" />
+          <cylinder length="${stretcher_mount_dist}" radius="0.007" />
         </geometry>
         <origin xyz="0 0 0" rpy="0 0 0" />
@@ -266,5 +266,5 @@
         <origin xyz="0 0 0" rpy="0 0 0" />
         <geometry>
-          <cylinder length="${stretcher_mount_dist}" radius="0.02" />
+          <cylinder length="${stretcher_mount_dist}" radius="0.007" />
         </geometry>
       </collision>
